Commit message: világ és turtlebot szerekesztés

File: robot_description/turtlebot3.urdf.xacro (robot description, xacro)
@@ -1,72 +1,70 @@
 <?xml version="1.0"?>
-<robot xmlns:xacro="http://ros.org/wiki/xacro" xmlns:ros="http://ros.org/wiki/ros">
-  <xacro:include filename="$(find turtlebot3_description)/urdf/turtlebot3.urdf.xacro"/>
-  <robot name="turtlebot3">
-    <xacro:property name="base_length" value="0.34"/>
-    <xacro:property name="base_width" value="0.34"/>
-    <xacro:property name="wheel_radius" value="0.1"/>
-    <xacro:property name="wheel_separation" value="0.2"/>
-    <link name="base_link">
-      <inertial>
-        <mass value="5.0"/>
-        <origin xyz="0 0 0.1" rpy="0 0 0"/>
-        <inertia ixx="0.1" ixy="0" ixz="0" iyy="0.1" iyz="0" izz="0.1"/>
-      </inertial>
-      <visual>
-        <geometry>
-          <box size="${base_length} ${base_width} 0.1"/>
-        </geometry>
-        <origin xyz="0 0 0.05" rpy="0 0 0"/>
-      </visual>
-      <collision>
-        <geometry>
-          <box size="${base_length} ${base_width} 0.1"/>
-        </geometry>
-        <origin xyz="0 0 0.05" rpy="0 0 0"/>
-      </collision>
-    </link>
-    <joint name="wheel_left_joint" type="revolute">
-      <parent link="base_link"/>
-      <child link="wheel_left"/>
-      <origin xyz="${wheel_separation/2} 0 0" rpy="0 0 0"/>
-      <axis xyz="0 0 1"/>
-      <limit effort="10" lower="-3.14" upper="3.14" velocity="1"/>
-    </joint>
-    <joint name="wheel_right_joint" type="revolute">
-      <parent link="base_link"/>
-      <child link="wheel_right"/>
-      <origin xyz="-${wheel_separation/2} 0 0" rpy="0 0 0"/>
-      <axis xyz="0 0 1"/>
-      <limit effort="10" lower="-3.14" upper="3.14" velocity="1"/>
-    </joint>
-    <link name="wheel_left">
-      <visual>
-        <geometry>
-          <cylinder radius="${wheel_radius}" length="0.1"/>
-        </geometry>
-        <origin xyz="${wheel_separation/2} 0 0" rpy="0 0 0"/>
-      </visual>
-      <collision>
-        <geometry>
-          <cylinder radius="${wheel_radius}" length="0.1"/>
-        </geometry>
-        <origin xyz="${wheel_separation/2} 0 0" rpy="0 0 0"/>
-      </collision>
-    </link>
-    <link name="wheel_right">
-      <visual>
-        <geometry>
-          <cylinder radius="${wheel_radius}" length="0.1"/>
-        </geometry>
-        <origin xyz="-${wheel_separation/2} 0 0" rpy="0 0 0"/>
-      </visual>
-      <collision>
-        <geometry>
-          <cylinder radius="${wheel_radius}" length="0.1"/>
-        </geometry>
-        <origin xyz="-${wheel_separation/2} 0 0" rpy="0 0 0"/>
-      </collision>
-    </link>
-    <xacro:include filename="$(find turtlebot3_description)/urdf/sensors.xacro"/>
-  </robot>
+<robot xmlns:xacro="http://ros.org/wiki/xacro" name="turtlebot3">
+  <xacro:property name="base_length" value="0.34"/>
+  <xacro:property name="base_width" value="0.34"/>
+  <xacro:property name="wheel_radius" value="0.1"/>
+  <xacro:property name="wheel_separation" value="0.2"/>
+  <link name="base_link">
+    <inertial>
+      <mass value="5.0"/>
+      <origin xyz="0 0 0.1" rpy="0 0 0"/>
+      <inertia ixx="0.1" ixy="0" ixz="0" iyy="0.1" iyz="0" izz="0.1"/>
+    </inertial>
+    <visual>
+      <geometry>
+        <box size="${base_length} ${base_width} 0.1"/>
+      </geometry>
+      <origin xyz="0 0 0.05" rpy="0 0 0"/>
+    </visual>
+    <collision>
+      <geometry>
+        <box size="${base_length} ${base_width} 0.1"/>
+      </geometry>
+      <origin xyz="0 0 0.05" rpy="0 0 0"/>
+    </collision>
+  </link>
+  <joint name="wheel_left_joint" type="revolute">
+    <parent link="base_link"/>
+    <child link="wheel_left"/>
+    <origin xyz="${wheel_separation/2} 0 0" rpy="0 0 0"/>
+    <axis xyz="0 0 1"/>
+    <limit effort="10" lower="-3.14" upper="3.14" velocity="1"/>
+  </joint>
+  <joint name="wheel_right_joint" type="revolute">
+    <parent link="base_link"/>
+    <child link="wheel_right"/>
+    <origin xyz="-${wheel_separation/2} 0 0" rpy="0 0 0"/>
+    <axis xyz="0 0 1"/>
+    <limit effort="10" lower="-3.14" upper="3.14" velocity="1"/>
+  </joint>
+  <link name="wheel_left">
+    <visual>
+      <geometry>
+        <cylinder radius="${wheel_radius}" length="0.1"/>
+      </geometry>
+      <origin xyz="0 0 0" rpy="0 0 0"/>
+    </visual>
+    <collision>
+      <geometry>
+        <cylinder radius="${wheel_radius}" length="0.1"/>
+      </geometry>
+      <origin xyz="0 0 0" rpy="0 0 0"/>
+    </collision>
+  </link>
+  <link name="wheel_right">
+    <visual>
+      <geometry>
+        <cylinder radius="${wheel_radius}" length="0.1"/>
+      </geometry>
+      <origin xyz="0 0 0" rpy="0 0 0"/>
+    </visual>
+    <collision>
+      <geometry>
+        <cylinder radius="${wheel_radius}" length="0.1"/>
+      </geometry>
+      <origin xyz="0 0 0" rpy="0 0 0"/>
+    </collision>
+  </link>
+  <!-- SENSORS NÉLKÜL! Ha kell, később bővítsd -->
+  <!-- <xacro:include filename="$(find turtlebot3_description)/urdf/sensors.xacro"/> -->
 </robot>

Commit message: parking logic szerkesztése

File: robot_description/turtlebot3.urdf.xacro (robot description, xacro)
@@ -28,5 +28,5 @@
     <child link="wheel_left"/>
     <origin xyz="${wheel_separation/2} 0 0" rpy="0 0 0"/>
-    <axis xyz="0 0 1"/>
+    <axis xyz="0 1 0"/>
     <limit effort="10" lower="-3.14" upper="3.14" velocity="1"/>
   </joint>
@@ -35,5 +35,5 @@
     <child link="wheel_right"/>
     <origin xyz="-${wheel_separation/2} 0 0" rpy="0 0 0"/>
-    <axis xyz="0 0 1"/>
+    <axis xyz="0 1 0"/>
     <limit effort="10" lower="-3.14" upper="3.14" velocity="1"/>
   </joint>
@@ -66,5 +66,19 @@
     </collision>
   </link>
-  <!-- SENSORS NÉLKÜL! Ha kell, később bővítsd -->
-  <!-- <xacro:include filename="$(find turtlebot3_description)/urdf/sensors.xacro"/> -->
+  <!-- Diff drive plugin hozzáadása -->
+  <gazebo>
+    <plugin name="diff_drive" filename="libgazebo_ros_diff_drive.so">
+      <ros>
+        <namespace>/</namespace>
+      </ros>
+      <update_rate>50</update_rate>
+      <left_wheel>wheel_left</left_wheel>
+      <right_wheel>wheel_right</right_wheel>
+      <wheel_separation>${wheel_separation}</wheel_separation>
+      <wheel_radius>${wheel_radius}</wheel_radius>
+      <command_topic>/cmd_vel</command_topic>
+      <odometry_topic>/odom</odometry_topic>
+      <publish_tf>true</publish_tf>
+    </plugin>
+  </gazebo>
 </robot>
