Commit message: robot és világ szerkesztése

File: robot_description/tb3_plain.urdf (robot description, URDF)
Before this commit: robot turtlebot3_burger, 7 links, 6 joints
Links:
- link base_link: geometry collision box size=0.140 0.140 0.143; visual mesh filename=file:///opt/ros/humble/share/turtlebot3_description/meshes/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 scale=0.001 0.001 0.001
- link base_scan: geometry collision cylinder length=0.0315 radius=0.055; visual mesh filename=file:///opt/ros/humble/share/turtlebot3_description/meshes/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 scale=0.001 0.001 0.001
- link wheel_left_link: geometry collision cylinder length=0.018 radius=0.033; visual mesh filename=file:///opt/ros/humble/share/turtlebot3_description/meshes/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 scale=0.001 0.001 0.001
- link wheel_right_link: geometry collision cylinder length=0.018 radius=0.033; visual mesh filename=file:///opt/ros/humble/share/turtlebot3_description/meshes/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 scale=0.001 0.001 0.001
